File: MotorCtrl.kicad_pcb (KiCad board)
At the start: 2 copper layers, 47 x 52.1 mm, 10 parts, among them J1 Conn_01x03_Female, J2 Conn_01x02_Female, J3 Conn_01x02_Female, Q1 BS108, Q2 IRLB8721PBF

Commit message: zones
Routing:
- added copper zone on F.Cu, net +12V
- added copper zone on F.Cu, net +5V
- added copper zone on F.Cu, net GND
- added copper zone on F.Cu, net Net-(D1-Pad2)
- added copper zone on F.Cu, net Net-(J1-Pad2)
- added copper zone on F.Cu, net Net-(R3-Pad2)
Changed lines of the file:
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@@
     (thickness 1.6)
   )
-  (paper "A4")
+  (paper "A5" portrait)
   (layers
     (0 "F.Cu" signal)
@@
       (psnegative false)
       (psa4output false)
-      (plotreference true)
+      (plotreference false)
       (plotvalue true)
       (plotinvisibletext false)
@@
       (subtractmaskfromsilk false)
       (outputformat 4)
-      (mirror true)
-      (drillshape 0)
+      (mirror false)
+      (drillshape 1)
       (scaleselection 1)
-      (outputdirectory "")
+      (outputdirectory "Exp/0/")
     )
   )
@@
   (segment (start 216.535 117.475) (end 216.535 126.04) (width 0.75) (layer "F.Cu") (net 8))
   (segment (start 218.71 117.475) (end 213.995 117.475) (width 0.75) (layer "F.Cu") (net 8))
+  (zone (net 7) (net_name "+5V") (layer "F.Cu") (hatch edge 0.508)
+    (connect_pads yes (clearance 0.508))
+    (min_thickness 0.254) (filled_areas_thickness no)
+    (fill yes (thermal_gap 0.508) (thermal_bridge_width 0.508) (island_removal_mode 1) (island_area_min 0))
+    (polygon
+      (pts
+        (xy 211.582 111.252)
+        (xy 205.232 111.252)
+        (xy 205.232 97.282)
+        (xy 211.582 97.282)
+      )
+    )
+  )
+  (zone (net 8) (net_name "Net-(R3-Pad2)") (layer "F.Cu") (hatch edge 0.508)
+    (connect_pads yes (clearance 0.508))
+    (min_thickness 0.254) (filled_areas_thickness no)
+    (fill yes (thermal_gap 0.508) (thermal_bridge_width 0.508))
+    (polygon
+      (pts
+        (xy 218.694 122.174)
+        (xy 217.17 122.174)
+        (xy 217.17 126.746)
+        (xy 213.868 126.746)
+        (xy 213.868 116.586)
+        (xy 218.694 116.586)
+      )
+    )
+  )
+  (zone (net 2) (net_name "Net-(D1-Pad2)") (layer "F.Cu") (hatch edge 0.508)
+    (connect_pads yes (clearance 0.508))
+    (min_thickness 0.254) (filled_areas_thickness no)
+    (fill yes (thermal_gap 0.508) (thermal_bridge_width 0.508) (smoothing fillet))
+    (polygon
+      (pts
+        (xy 210.82 128.778)
+        (xy 219.964 128.778)
+        (xy 219.964 129.794)
+        (xy 217.932 131.826)
+        (xy 217.932 135.128)
+        (xy 209.296 135.128)
+        (xy 207.518 133.096)
+        (xy 200.66 133.096)
+        (xy 200.66 127.254)
+        (xy 208.28 127.254)
+      )
+    )
+  )
+  (zone (net 1) (net_name "+12V") (layer "F.Cu") (hatch edge 0.508)
+    (connect_pads yes (clearance 0.508))
+    (min_thickness 0.254) (filled_areas_thickness no)
+    (fill yes (thermal_gap 0.508) (thermal_bridge_width 0.508) (island_removal_mode 1) (island_area_min 0))
+    (polygon
+      (pts
+        (xy 212.09 118.872)
+        (xy 199.136 118.872)
+        (xy 199.136 135.636)
+        (xy 206.248 135.636)
+        (xy 206.248 136.652)
+        (xy 220.726 136.652)
+        (xy 220.726 131.064)
+        (xy 233.172 131.064)
+        (xy 233.172 138.176)
+        (xy 230.632 139.446)
+        (xy 229.616 142.24)
+        (xy 200.914 142.24)
+        (xy 200.914 138.938)
+        (xy 197.104 138.938)
+        (xy 197.104 116.078)
+        (xy 212.09 116.078)
+      )
+    )
+  )
+  (zone (net 6) (net_name "Net-(J1-Pad2)") (layer "F.Cu") (hatch edge 0.508)
+    (connect_pads yes (clearance 0.508))
+    (min_thickness 0.254) (filled_areas_thickness no)
+    (fill yes (thermal_gap 0.508) (thermal_bridge_width 0.508) (island_removal_mode 1) (island_area_min 0))
+    (polygon
+      (pts
+        (xy 220.472 111.76)
+        (xy 214.122 111.76)
+        (xy 214.122 97.282)
+        (xy 220.472 97.282)
+      )
+    )
+  )
+  (zone (net 5) (net_name "GND") (layer "F.Cu") (hatch edge 0.508)
+    (connect_pads yes (clearance 0.508))
+    (min_thickness 0.254) (filled_areas_thickness no)
+    (fill yes (thermal_gap 0.508) (thermal_bridge_width 0.508))
+    (polygon
+      (pts
+        (xy 233.170805 127.761913)
+        (xy 221.487986 127.762006)
+        (xy 221.488 121.92)
+        (xy 228.346 121.92)
+        (xy 228.346 111.252)
+        (xy 223.266 111.252)
+        (xy 223.266 97.282)
+        (xy 228.6 97.282)
+        (xy 228.6 105.399865)
+        (xy 233.171507 105.389729)
+      )
+    )
+  )
 )

Commit message: ff
Parts:
- moved J1 246.1 mm to (25.3, 248.5), turned to -90 degrees
- moved R1 235.0 mm to (31.9, 257.3), turned to 180 degrees
- moved R2 234.2 mm to (31.6, 266.2), turned to 0 degrees
- moved Q1 233.9 mm to (34.0, 248.4), turned to 90 degrees
- moved R4 228.8 mm to (36.7, 254.8), turned to 90 degrees
- moved R3 227.6 mm to (36.7, 261.5), turned to 90 degrees
- moved Q2 216.2 mm to (45.3, 257.9), turned to 90 degrees
- moved J2 207.2 mm to (53.8, 245.9), turned to 180 degrees
- moved D1 206.1 mm to (53.2, 252.9), turned to -90 degrees
- moved J3 196.2 mm to (58.3, 271.3), turned to 180 degrees
Other:
- board size 47 x 52.1 mm -> 52.1 x 47 mm

Commit message: round
Parts:
- moved J1 29.2 mm to (54.0, 243.6), turned to 180 degrees
- moved J3 27.6 mm to (31.2, 276.6), turned to 90 degrees
- moved J2 26.4 mm to (56.6, 272.1), turned to 90 degrees
- moved Q1 20.4 mm to (54.1, 252.3), turned to 0 degrees
- moved D1 19.0 mm to (49.7, 271.5), turned to 180 degrees
- moved R2 17.0 mm to (36.3, 249.9), turned to -90 degrees
- moved R1 15.1 mm to (45.2, 250.2), turned to 90 degrees
- moved R4 11.1 mm to (47.8, 255.0), turned to 0 degrees
- moved R3 7.81 mm to (41.0, 255.0), turned to 0 degrees
- moved Q2 5.65 mm to (44.6, 263.5), turned to 0 degrees
Routing:
- net +12V: track 71.5 -> 67.2 mm
- net Net-(D1-Pad2): track 23.9 -> 22.5 mm
- net Net-(Q1-Pad2): track 19.2 -> 20.1 mm
Other:
- board size 52.1 x 47 mm -> 47 x 52.1 mm
